Commit message: up

File: src/puppy_description/urdf/puppy.gazebo.xacro (robot description, xacro)
@@ -4,33 +4,39 @@
     <plugin name="gazebo_ros_control" filename="libgazebo_ros_control.so">
       <robotNamespace>/puppy</robotNamespace>
+      <robotSimType>gazebo_ros_control/DefaultRobotHWSim</robotSimType>
+      <legacyModeNS>true</legacyModeNS>
     </plugin>
   </gazebo>
-  <gazebo reference="lf_link2">
+  <xacro:macro name="joint_setup_block" params="joint_name">
+    <gazebo reference="${joint_name}">
+      <implicitSpringDamper>1</implicitSpringDamper>
+    </gazebo>
+  </xacro:macro>
+  <xacro:joint_setup_block joint_name="lf_joint1"/>
+  <xacro:joint_setup_block joint_name="lf_joint2"/>
+  <xacro:joint_setup_block joint_name="rf_joint1"/>
+  <xacro:joint_setup_block joint_name="rf_joint2"/>
+  <xacro:joint_setup_block joint_name="lb_joint1"/>
+  <xacro:joint_setup_block joint_name="lb_joint2"/>
+  <xacro:joint_setup_block joint_name="rb_joint1"/>
+  <xacro:joint_setup_block joint_name="rb_joint2"/>
+  <xacro:macro name="link_setup_block" params="link_name">
+    <gazebo reference="${link_name}">
+      <kp>1000000.0</kp>
+      <kd>1.0</kd>
+      <mu1>0.6</mu1>
+      <mu2>0.6</mu2>
+      <minDepth>0.001</minDepth>
+    </gazebo>
+  </xacro:macro>
+  <xacro:link_setup_block link_name="lf_link2"/>
+  <xacro:link_setup_block link_name="rf_link2"/>
+  <xacro:link_setup_block link_name="lb_link2"/>
+  <xacro:link_setup_block link_name="rb_link2"/>
+  <!--gazebo reference="lf_link2">
     <mu1>1.0</mu1>
     <mu2>1.0</mu2>
     <minDepth>0.0002</minDepth>
     <kp  value="1000000.0"/>
-    <kd  value="100.0"/>
-  </gazebo>
-  <gazebo reference="rf_link2">
-    <mu1>1.0</mu1>
-    <mu2>1.0</mu2>
-    <minDepth>0.0002</minDepth>
-    <kp  value="1000000.0"/>
-    <kd  value="100.0"/>
-  </gazebo>
-  <gazebo reference="lb_link2">
-    <mu1>1.0</mu1>
-    <mu2>1.0</mu2>
-    <minDepth>0.0002</minDepth>
-    <kp  value="1000000.0"/>
-    <kd  value="100.0"/>
-  </gazebo>
-  <gazebo reference="rb_link2">
-    <mu1>1.0</mu1>
-    <mu2>1.0</mu2>
-    <minDepth>0.0002</minDepth>
-    <kp  value="1000000.0"/>
-    <kd  value="100.0"/>
-  </gazebo>
+    <kd  value="100.0"/-->
 </robot>

File: src/puppy_description/urdf/puppy.urdf.xacro (robot description, xacro)
@@ -3,6 +3,6 @@
   <xacro:include filename="$(find puppy_description)/urdf/puppy.transmission.xacro"/>
   <xacro:include filename="$(find puppy_description)/urdf/puppy.gazebo.xacro"/>
-  <xacro:property name="motor_torque" value="0.1"/>
-  <xacro:property name="motor_vec" value="0.1"/>
+  <xacro:property name="motor_torque" value="1.4"/>
+  <xacro:property name="motor_vec" value="2"/>
   <link name="base_footprint" />
   <joint name="base_joint" type="fixed">
@@ -96,5 +96,5 @@
     <origin
       xyz="0.0420105649539 0.0778693100523862 0.0159880060021007"
-      rpy="-0.766 0 0" />
+      rpy="-0.752 0 0" />
     <parent
       link="base_link" />
@@ -212,5 +212,5 @@
     <origin
       xyz="-0.0420105649534512 0.0778693100523859 0.0159880060091649"
-      rpy="-0.766 0 0" />
+      rpy="-0.752 0 0" />
     <parent
       link="base_link" />
@@ -328,5 +328,5 @@
     <origin
       xyz="-0.0420105469986279 -0.0778692767711234 0.0106512951143373"
-      rpy="-0.766 0 0" />
+      rpy="-0.752 0 0" />
     <parent
       link="base_link" />
@@ -444,5 +444,5 @@
     <origin
       xyz="0.0420105469981795 -0.0778692767711239 0.0106512951072731"
-      rpy="-0.766 0 0" />
+      rpy="-0.752 0 0" />
     <parent
       link="base_link" />

File: src/puppy_description/urdf_bk/puppy.urdf.xacro (robot description, xacro)
@@ -98,5 +98,5 @@
     <origin
       xyz="0.0420105649539 0.0778693100523862 0.0159880060021007"
-      rpy="0.8342537604318887 0 0" />
+      rpy="0.0342537604318887 0 0" />
     <parent
       link="base_link" />

Commit message: finish simple move

File: src/puppy_description/urdf/puppy.gazebo.xacro (robot description, xacro)
@@ -8,5 +8,5 @@
     </plugin>
   </gazebo>
-  <xacro:macro name="joint_setup_block" params="joint_name">
+  <!--xacro:macro name="joint_setup_block" params="joint_name">
     <gazebo reference="${joint_name}">
       <implicitSpringDamper>1</implicitSpringDamper>
@@ -20,12 +20,12 @@
   <xacro:joint_setup_block joint_name="lb_joint2"/>
   <xacro:joint_setup_block joint_name="rb_joint1"/>
-  <xacro:joint_setup_block joint_name="rb_joint2"/>
+  <xacro:joint_setup_block joint_name="rb_joint2"/-->
   <xacro:macro name="link_setup_block" params="link_name">
     <gazebo reference="${link_name}">
       <kp>1000000.0</kp>
       <kd>1.0</kd>
-      <mu1>0.6</mu1>
-      <mu2>0.6</mu2>
-      <minDepth>0.001</minDepth>
+      <mu1>0.05</mu1>
+      <mu2>0.05</mu2>
+      <minDepth>0.0002</minDepth>
     </gazebo>
   </xacro:macro>

File: src/puppy_description/urdf/puppy.urdf.xacro (robot description, xacro)
@@ -3,6 +3,6 @@
   <xacro:include filename="$(find puppy_description)/urdf/puppy.transmission.xacro"/>
   <xacro:include filename="$(find puppy_description)/urdf/puppy.gazebo.xacro"/>
-  <xacro:property name="motor_torque" value="1.4"/>
-  <xacro:property name="motor_vec" value="2"/>
+  <xacro:property name="motor_torque" value="0.1"/>
+  <xacro:property name="motor_vec" value="1"/>
   <link name="base_footprint" />
   <joint name="base_joint" type="fixed">

Commit message: up

File: src/puppy_description/urdf/puppy.gazebo.xacro (robot description, xacro)
@@ -25,13 +25,13 @@
       <kp>1000000.0</kp>
       <kd>1.0</kd>
-      <mu1>0.05</mu1>
-      <mu2>0.05</mu2>
+      <mu1>0.3</mu1>
+      <mu2>0.3</mu2>
       <minDepth>0.0002</minDepth>
     </gazebo>
   </xacro:macro>
-  <xacro:link_setup_block link_name="lf_link2"/>
-  <xacro:link_setup_block link_name="rf_link2"/>
-  <xacro:link_setup_block link_name="lb_link2"/>
-  <xacro:link_setup_block link_name="rb_link2"/>
+  <xacro:link_setup_block link_name="lf_link3"/>
+  <xacro:link_setup_block link_name="rf_link3"/>
+  <xacro:link_setup_block link_name="lb_link3"/>
+  <xacro:link_setup_block link_name="rb_link3"/>
   <!--gazebo reference="lf_link2">
     <mu1>1.0</mu1>

File: src/puppy_description/urdf/puppy.urdf.xacro (robot description, xacro)
@@ -3,11 +3,12 @@
   <xacro:include filename="$(find puppy_description)/urdf/puppy.transmission.xacro"/>
   <xacro:include filename="$(find puppy_description)/urdf/puppy.gazebo.xacro"/>
-  <xacro:property name="motor_torque" value="0.1"/>
-  <xacro:property name="motor_vec" value="1"/>
+  <xacro:include filename="materials.xacro" />
+  <xacro:property name="motor_torque" value="0.5"/>
+  <xacro:property name="motor_vec" value="2"/>
   <link name="base_footprint" />
   <joint name="base_joint" type="fixed">
     <parent link="base_footprint" />
     <child link="base_link" />
-    <origin xyz="0.0 0.0 0.109" rpy="0 0 0" />
+    <origin xyz="0.0 0.0 0.11" rpy="0 0 0" />
   </joint>
   <link
@@ -36,7 +37,5 @@
       </geometry>
       <material
-        name="">
-        <color
-          rgba="1 1 1 1" />
+        name="black">
       </material>
     </visual>
@@ -76,7 +75,5 @@
       </geometry>
       <material
-        name="">
-        <color
-          rgba="0.752941176470588 0.752941176470588 0.752941176470588 1" />
+        name="black">
       </material>
     </visual>
@@ -134,7 +131,5 @@
       </geometry>
       <material
-        name="">
-        <color
-          rgba="0.752941176470588 0.752941176470588 0.752941176470588 1" />
+        name="black">
       </material>
     </visual>
@@ -192,7 +187,5 @@
       </geometry>
       <material
-        name="">
-        <color
-          rgba="0.752941176470588 0.752941176470588 0.752941176470588 1" />
+        name="black">
       </material>
     </visual>
@@ -250,7 +243,5 @@
       </geometry>
       <material
-        name="">
-        <color
-          rgba="0.752941176470588 0.752941176470588 0.752941176470588 1" />
+        name="black">
       </material>
     </visual>
@@ -308,7 +299,5 @@
       </geometry>
       <material
-        name="">
-        <color
-          rgba="0.752941176470588 0.752941176470588 0.752941176470588 1" />
+        name="black">
       </material>
     </visual>
@@ -366,7 +355,5 @@
       </geometry>
       <material
-        name="">
-        <color
-          rgba="0.752941176470588 0.752941176470588 0.752941176470588 1" />
+        name="black">
       </material>
     </visual>
@@ -424,7 +411,5 @@
       </geometry>
       <material
-        name="">
-        <color
-          rgba="0.752941176470588 0.752941176470588 0.752941176470588 1" />
+        name="black">
       </material>
     </visual>
@@ -482,7 +467,5 @@
       </geometry>
       <material
-        name="">
-        <color
-          rgba="0.752941176470588 0.752941176470588 0.752941176470588 1" />
+        name="black">
       </material>
     </visual>
@@ -540,7 +523,5 @@
       </geometry>
       <material
-        name="">
-        <color
-          rgba="0.752941176470588 0.752941176470588 0.752941176470588 1" />
+        name="black">
       </material>
     </visual>
@@ -568,3 +549,147 @@
       xyz="0 0 0" />
   </joint>
+  <link name="lf_link3">
+    <inertial>
+      <origin
+        xyz="0 0 0"
+        rpy="0 0 0" />
+     <mass
+        value="0.0391" />
+      <inertia
+        ixx="3.7713E-012"
+        ixy="0"
+        ixz="0"
+        iyy="3.5422E-12"
+        iyz="0"
+        izz="5.443E-012" />
+    </inertial>
+    <collision>
+      <origin
+        xyz="0.0032 0 0.001"
+        rpy="0 1.57 0" />
+      <geometry>
+        <cylinder radius="0.01" length="0.01"/>
+      </geometry>
+    </collision>
+  </link>
+  <link name="rf_link3">
+    <inertial>
+      <origin
+        xyz="0 0 0"
+        rpy="0 0 0" />
+     <mass
+        value="0.0391" />
+      <inertia
+        ixx="3.7713E-012"
+        ixy="0"
+        ixz="0"
+        iyy="3.5422E-12"
+        iyz="0"
+        izz="5.443E-012" />
+    </inertial>
+    <collision>
+      <origin
+        xyz="0.0032 0 0.001"
+        rpy="0 1.57 0" />
+      <geometry>
+        <cylinder radius="0.01" length="0.01"/>
+      </geometry>
+    </collision>
+  </link>
+  <link name="lb_link3">
+    <inertial>
+      <origin
+        xyz="0 0 0"
+        rpy="0 0 0" />
+     <mass
+        value="0.0391" />
+      <inertia
+        ixx="3.7713E-012"
+        ixy="0"
+        ixz="0"
+        iyy="3.5422E-12"
+        iyz="0"
+        izz="5.443E-012" />
+    </inertial>
+    <collision>
+      <origin
+        xyz="0.0032 0 0.001"
+        rpy="0 1.57 0" />
+      <geometry>
+        <cylinder radius="0.01" length="0.01"/>
+      </geometry>
+    </collision>
+  </link>
+  <link name="rb_link3">
+    <inertial>
+      <origin
+        xyz="0 0 0"
+        rpy="0 0 0" />
+     <mass
+        value="0.0391" />
+      <inertia
+        ixx="3.7713E-012"
+        ixy="0"
+        ixz="0"
+        iyy="3.5422E-12"
+        iyz="0"
+        izz="5.443E-012" />
+    </inertial>
+    <collision>
+      <origin
+        xyz="0.0032 0 0.001"
+        rpy="0 1.57 0" />
+      <geometry>
+        <cylinder radius="0.01" length="0.01"/>
+      </geometry>
+    </collision>
+  </link>
+  <joint name="lf_joint3"
+    type="fixed">
+    <origin
+      xyz="0 -0.053 -0.053"
+      rpy="0.78 0 0" />
+    <parent
+      link="lf_link2" />
+    <child
+      link="lf_link3" />
+    <axis
+      xyz="0 0 0" />
+  </joint>
+  <joint name="rf_joint3"
+    type="fixed">
+    <origin
+      xyz="0 -0.053 -0.053"
+      rpy="0.78 0 0" />
+    <parent
+      link="rf_link2" />
+    <child
+      link="rf_link3" />
+    <axis
+      xyz="0 0 0" />
+  </joint>
+  <joint name="lb_joint3"
+    type="fixed">
+    <origin
+      xyz="0 -0.053 -0.053"
+      rpy="0.78 0 0" />
+    <parent
+      link="lb_link2" />
+    <child
+      link="lb_link3" />
+    <axis
+      xyz="0 0 0" />
+  </joint>
+  <joint name="rb_joint3"
+    type="fixed">
+    <origin
+      xyz="0 -0.053 -0.053"
+      rpy="0.78 0 0" />
+    <parent
+      link="rb_link2" />
+    <child
+      link="rb_link3" />
+    <axis
+      xyz="0 0 0" />
+  </joint>
 </robot>

Commit message: up

File: src/puppy_description/urdf/puppy.gazebo.xacro (robot description, xacro)
@@ -25,6 +25,6 @@
       <kp>1000000.0</kp>
       <kd>1.0</kd>
-      <mu1>0.3</mu1>
-      <mu2>0.3</mu2>
+      <mu1>0.8</mu1>
+      <mu2>0.8</mu2>
       <minDepth>0.0002</minDepth>
     </gazebo>

File: src/puppy_description/urdf/puppy.urdf.xacro (robot description, xacro)
@@ -4,5 +4,5 @@
   <xacro:include filename="$(find puppy_description)/urdf/puppy.gazebo.xacro"/>
   <xacro:include filename="materials.xacro" />
-  <xacro:property name="motor_torque" value="0.5"/>
+  <xacro:property name="motor_torque" value="1"/>
   <xacro:property name="motor_vec" value="2"/>
   <link name="base_footprint" />

Commit message: finish

File: src/puppy_description/urdf/puppy.gazebo.xacro (robot description, xacro)
@@ -21,10 +21,30 @@
   <xacro:joint_setup_block joint_name="rb_joint1"/>
   <xacro:joint_setup_block joint_name="rb_joint2"/-->
+  <xacro:macro name="model_color" params="link_name">
+    <gazebo reference="${link_name}">
+      <material>Gazebo/Black</material>
+      <turnGravityOff>false</turnGravityOff>
+    </gazebo>
+  </xacro:macro>
+  <xacro:model_color link_name="base_link"/>
+  <xacro:model_color link_name="lf_link1"/>
+  <xacro:model_color link_name="lf_link2"/>
+  <xacro:model_color link_name="lf_link3"/>
+  <xacro:model_color link_name="rf_link1"/>
+  <xacro:model_color link_name="rf_link2"/>
+  <xacro:model_color link_name="rf_link3"/>
+  <xacro:model_color link_name="lb_link1"/>
+  <xacro:model_color link_name="lb_link2"/>
+  <xacro:model_color link_name="lb_link3"/>
+  <xacro:model_color link_name="rb_link1"/>
+  <xacro:model_color link_name="rb_link2"/>
+  <xacro:model_color link_name="rb_link3"/>
+  <xacro:model_color link_name="camera_link"/>
   <xacro:macro name="link_setup_block" params="link_name">
     <gazebo reference="${link_name}">
       <kp>1000000.0</kp>
       <kd>1.0</kd>
-      <mu1>0.8</mu1>
-      <mu2>0.8</mu2>
+      <mu1>0.4</mu1>
+      <mu2>0.4</mu2>
       <minDepth>0.0002</minDepth>
     </gazebo>

File: src/puppy_description/urdf/puppy.urdf.xacro (robot description, xacro)
@@ -4,5 +4,5 @@
   <xacro:include filename="$(find puppy_description)/urdf/puppy.gazebo.xacro"/>
   <xacro:include filename="materials.xacro" />
-  <xacro:property name="motor_torque" value="1"/>
+  <xacro:property name="motor_torque" value="0.5"/>
   <xacro:property name="motor_vec" value="2"/>
   <link name="base_footprint" />
@@ -569,5 +569,5 @@
         rpy="0 1.57 0" />
       <geometry>
-        <cylinder radius="0.01" length="0.01"/>
+        <cylinder radius="0.0095" length="0.01"/>
       </geometry>
     </collision>
@@ -593,5 +593,5 @@
         rpy="0 1.57 0" />
       <geometry>
-        <cylinder radius="0.01" length="0.01"/>
+        <cylinder radius="0.0095" length="0.01"/>
       </geometry>
     </collision>
@@ -617,5 +617,5 @@
         rpy="0 1.57 0" />
       <geometry>
-        <cylinder radius="0.01" length="0.01"/>
+        <cylinder radius="0.0095" length="0.01"/>
       </geometry>
     </collision>
@@ -641,5 +641,5 @@
         rpy="0 1.57 0" />
       <geometry>
-        <cylinder radius="0.01" length="0.01"/>
+        <cylinder radius="0.0095" length="0.01"/>
       </geometry>
     </collision>

Commit message: first push

File: src/puppy_description/urdf/puppy.gazebo.xacro (robot description, xacro)
@@ -8,17 +8,4 @@
     </plugin>
   </gazebo>
-  <!--xacro:macro name="joint_setup_block" params="joint_name">
-    <gazebo reference="${joint_name}">
-      <implicitSpringDamper>1</implicitSpringDamper>
-    </gazebo>
-  </xacro:macro>
-  <xacro:joint_setup_block joint_name="lf_joint1"/>
-  <xacro:joint_setup_block joint_name="lf_joint2"/>
-  <xacro:joint_setup_block joint_name="rf_joint1"/>
-  <xacro:joint_setup_block joint_name="rf_joint2"/>
-  <xacro:joint_setup_block joint_name="lb_joint1"/>
-  <xacro:joint_setup_block joint_name="lb_joint2"/>
-  <xacro:joint_setup_block joint_name="rb_joint1"/>
-  <xacro:joint_setup_block joint_name="rb_joint2"/-->
   <xacro:macro name="model_color" params="link_name">
     <gazebo reference="${link_name}">
@@ -54,9 +41,3 @@
   <xacro:link_setup_block link_name="lb_link3"/>
   <xacro:link_setup_block link_name="rb_link3"/>
-  <!--gazebo reference="lf_link2">
-    <mu1>1.0</mu1>
-    <mu2>1.0</mu2>
-    <minDepth>0.0002</minDepth>
-    <kp  value="1000000.0"/>
-    <kd  value="100.0"/-->
 </robot>

File: src/puppy_description/urdf/puppy.urdf.xacro (robot description, xacro)
@@ -12,6 +12,12 @@
     <origin xyz="0.0 0.0 0.11" rpy="0 0 0" />
   </joint>
-  <link
-    name="base_link">
+  <link name="base_link" />
+  <joint name="dummy_joint" type="fixed">
+    <parent link="base_link" />
+    <child link="base_dummy" />
+    <origin xyz="0.0 0.0 0.0" rpy="0 0 1.57" />
+  </joint>
+  <link
+    name="base_dummy">
     <inertial>
       <origin
@@ -20,4 +26,7 @@
       <mass
         value="0.0656002451111466" />
+      <material
+        name="black">
+      </material>
       <inertia
         ixx="0.0001015640290354"
@@ -95,5 +104,5 @@
       rpy="-0.752 0 0" />
     <parent
-      link="base_link" />
+      link="base_dummy" />
     <child
       link="lb_link1" />
@@ -207,5 +216,5 @@
       rpy="-0.752 0 0" />
     <parent
-      link="base_link" />
+      link="base_dummy" />
     <child
       link="rb_link1" />
@@ -319,5 +328,5 @@
       rpy="-0.752 0 0" />
     <parent
-      link="base_link" />
+      link="base_dummy" />
     <child
       link="rf_link1" />
@@ -431,5 +440,5 @@
       rpy="-0.752 0 0" />
     <parent
-      link="base_link" />
+      link="base_dummy" />
     <child
       link="lf_link1" />
@@ -543,5 +552,5 @@
       rpy="0.0342537604318887 0 0" />
     <parent
-      link="base_link" />
+      link="base_dummy" />
     <child
       link="camera_link" />
