Commit message: defined additional colors

File: src/puppy_description/urdf/materials.xacro (robot description, xacro)
@@ -2,20 +2,20 @@
 <robot>
   <material name="black">
-    <color rgba="0.0 0.0 0.0 1.0"/>
+    <color rgba="1.0 1.0 1.0 1.0"/>
   </material>
   <material name="blue">
-    <color rgba="0.0 0.0 0.8 1.0"/>
+    <color rgba="1.0 1.0 1.0 1.0"/>
   </material>
   <material name="green">
-    <color rgba="0.0 0.8 0.0 1.0"/>
+    <color rgba="1.0 1.0 1.0 1.0"/>
   </material>
   <material name="gray">
-    <color rgba="0.7 0.7 0.7 1.0"/>
+    <color rgba="1.0 1.0 1.0 1.0"/>
   </material>
   <material name="darkgray">
-    <color rgba="0.3 0.3 0.3 1.0"/>
+    <color rgba="1.0 1.0 1.0 1.0"/>
   </material>
   <material name="red">
-    <color rgba="0.8 0.0 0.0 1.0"/>
+    <color rgba="1.0 1.0 1.0 1.0"/>
   </material>
   <material name="white">
@@ -23,5 +23,8 @@
   </material>
   <material name="yellow">
-    <color rgba="0.8 0.8 0.0 1.0"/>
+    <color rgba="1.0 1.0 1.0 1.0"/>
+  </material>
+  <material name="grey">
+    <color rgba="1.0 1.0 1.0 1.0"/>
   </material>
 </robot>
