Commit message: restructure positional coordinates

File: src/puppy_description/urdf/puppy.urdf.xacro (robot description, xacro)
@@ -12,48 +12,22 @@
     <origin xyz="0.0 0.0 0.11" rpy="0 0 0" />
   </joint>
-  <link name="base_link" />
-  <joint name="dummy_joint" type="fixed">
-    <parent link="base_link" />
-    <child link="base_dummy" />
-    <origin xyz="0.0 0.0 0.0" rpy="0 0 1.57" />
-  </joint>
-  <link
-    name="base_dummy">
-    <inertial>
-      <origin
-        xyz="-0.000281314271092793 -0.00232093824972492 0.0187442604423227"
-        rpy="0 0 0" />
-      <mass
-        value="0.0656002451111466" />
-      <material
-        name="black">
-      </material>
-      <inertia
-        ixx="0.0001015640290354"
-        ixy="5.44665608405109E-10"
-        ixz="-5.74905560030545E-09"
-        iyy="4.73014549137098E-05"
-        iyz="-4.46099046853099E-06"
-        izz="0.000137571042581761" />
-    </inertial>
-    <visual>
-      <origin
-        xyz="0 0 0"
-        rpy="0 0 0" />
-      <geometry>
-        <mesh
-          filename="package://puppy_description/meshes/base_link.STL" />
-      </geometry>
-      <material
-        name="black">
-      </material>
-    </visual>
-    <collision>
-      <origin
-        xyz="0 0 0"
-        rpy="0 0 0" />
-      <geometry>
-        <mesh
-          filename="package://puppy_description/meshes/base_link.STL" />
+  <link name="base_link">
+    <inertial>
+      <origin xyz="-0.000281314271092793 -0.00232093824972492 0.0187442604423227" rpy="0 0 0"/>
+      <mass value="0.0656002451111466"/>
+      <inertia ixx="0.0001015640290354" ixy="5.44665608405109E-10" ixz="-5.74905560030545E-09"
+               iyy="4.73014549137098E-05" iyz="-4.46099046853099E-06" izz="0.000137571042581761"/>
+    </inertial>
+    <visual>
+      <origin xyz="0 0 0" rpy="0 0 0"/>
+      <geometry>
+        <mesh filename="package://puppy_description/meshes/base_link.STL"/>
+      </geometry>
+      <material name="black"/>
+    </visual>
+    <collision>
+      <origin xyz="0 0 0" rpy="0 0 0"/>
+      <geometry>
+        <mesh filename="package://puppy_description/meshes/base_link.STL"/>
       </geometry>
     </collision>
@@ -101,8 +75,8 @@
     type="revolute">
     <origin
-      xyz="0.0420105649539 0.0778693100523862 0.0159880060021007"
+      xyz="0.042 0.078 0.016"
       rpy="-0.752 0 0" />
     <parent
-      link="base_dummy" />
+      link="base_link" />
     <child
       link="lb_link1" />
@@ -111,5 +85,5 @@
     <limit
       lower="-2"
-      upper=" 2"
+      upper="2"
       effort="${motor_torque}"
       velocity="${motor_vec}" />
@@ -157,5 +131,5 @@
     type="revolute">
     <origin
-      xyz="0.0120498902789596 0.0525235728370777 -0.052877465200695"
+      xyz="0.012 0.053 -0.053"
       rpy="0 0 0" />
     <parent
@@ -213,8 +187,8 @@
     type="revolute">
     <origin
-      xyz="-0.0420105649534512 0.0778693100523859 0.0159880060091649"
+      xyz="-0.042 0.078 0.016"
       rpy="-0.752 0 0" />
     <parent
-      link="base_dummy" />
+      link="base_link" />
     <child
       link="rb_link1" />
@@ -269,5 +243,5 @@
     type="revolute">
     <origin
-      xyz="-0.0185498902789654 0.0525235728370851 -0.0528774652006949"
+      xyz="-0.019 0.053 -0.053"
       rpy="0 0 0" />
     <parent
@@ -325,8 +299,8 @@
     type="revolute">
     <origin
-      xyz="-0.0420105469986279 -0.0778692767711234 0.0106512951143373"
+      xyz="-0.042 -0.078 0.011"
       rpy="-0.752 0 0" />
     <parent
-      link="base_dummy" />
+      link="base_link" />
     <child
       link="rf_link1" />
@@ -381,5 +355,5 @@
     type="revolute">
     <origin
-      xyz="-0.0185498902789602 0.0525235728370692 -0.0528774652007036"
+      xyz="-0.019 0.053 -0.053"
       rpy="0 0 0" />
     <parent
@@ -437,8 +411,8 @@
     type="revolute">
     <origin
-      xyz="0.0420105469981795 -0.0778692767711239 0.0106512951072731"
+      xyz="0.042 -0.078 0.011"
       rpy="-0.752 0 0" />
     <parent
-      link="base_dummy" />
+      link="base_link" />
     <child
       link="lf_link1" />
@@ -493,5 +467,5 @@
     type="revolute">
     <origin
-      xyz="0.0120498902789604 0.0525235728370695 -0.0528774652007036"
+      xyz="0.012 0.053 -0.053"
       rpy="0 0 0" />
     <parent
@@ -552,5 +526,5 @@
       rpy="0.0342537604318887 0 0" />
     <parent
-      link="base_dummy" />
+      link="base_link" />
     <child
       link="camera_link" />

Commit message: change color to white

File: src/puppy_description/urdf/puppy.urdf.xacro (robot description, xacro)
@@ -24,5 +24,5 @@
         <mesh filename="package://puppy_description/meshes/base_link.STL"/>
       </geometry>
-      <material name="black"/>
+      <material name="white"/>
     </visual>
     <collision>
@@ -33,4 +33,15 @@
     </collision>
   </link>
+  <!-- Gazebo override for base_link -->
+  <gazebo reference="base_link">
+    <visual>
+      <material>
+        <ambient>1 1 1 1</ambient>
+        <diffuse>1 1 1 1</diffuse>
+        <specular>1 1 1 1</specular>
+        <emissive>0 0 0 1</emissive>
+      </material>
+    </visual>
+  </gazebo>
   <link
     name="lb_link1">
@@ -58,5 +69,5 @@
       </geometry>
       <material
-        name="black">
+        name="white">
       </material>
     </visual>
@@ -71,4 +82,14 @@
     </collision>
   </link>
+  <gazebo reference="lb_link1">
+    <visual>
+      <material>
+        <ambient>1 1 1 1</ambient>
+        <diffuse>1 1 1 1</diffuse>
+        <specular>1 1 1 1</specular>
+        <emissive>0 0 0 1</emissive>
+      </material>
+    </visual>
+  </gazebo>
   <joint
     name="lb_joint1"
@@ -114,5 +135,5 @@
       </geometry>
       <material
-        name="black">
+        name="white">
       </material>
     </visual>
@@ -127,4 +148,14 @@
     </collision>
   </link>
+  <gazebo reference="lb_link2">
+    <visual>
+      <material>
+        <ambient>1 1 1 1</ambient>
+        <diffuse>1 1 1 1</diffuse>
+        <specular>1 1 1 1</specular>
+        <emissive>0 0 0 1</emissive>
+      </material>
+    </visual>
+  </gazebo>
   <joint
     name="lb_joint2"
@@ -170,5 +201,5 @@
       </geometry>
       <material
-        name="black">
+        name="white">
       </material>
     </visual>
@@ -183,4 +214,14 @@
     </collision>
   </link>
+  <gazebo reference="rb_link1">
+    <visual>
+      <material>
+        <ambient>1 1 1 1</ambient>
+        <diffuse>1 1 1 1</diffuse>
+        <specular>1 1 1 1</specular>
+        <emissive>0 0 0 1</emissive>
+      </material>
+    </visual>
+  </gazebo>
   <joint
     name="rb_joint1"
@@ -226,5 +267,5 @@
       </geometry>
       <material
-        name="black">
+        name="white">
       </material>
     </visual>
@@ -239,4 +280,14 @@
     </collision>
   </link>
+  <gazebo reference="rb_link2">
+    <visual>
+      <material>
+        <ambient>1 1 1 1</ambient>
+        <diffuse>1 1 1 1</diffuse>
+        <specular>1 1 1 1</specular>
+        <emissive>0 0 0 1</emissive>
+      </material>
+    </visual>
+  </gazebo>
   <joint
     name="rb_joint2"
@@ -282,5 +333,5 @@
       </geometry>
       <material
-        name="black">
+        name="white">
       </material>
     </visual>
@@ -295,4 +346,14 @@
     </collision>
   </link>
+  <gazebo reference="rf_link1">
+    <visual>
+      <material>
+        <ambient>1 1 1 1</ambient>
+        <diffuse>1 1 1 1</diffuse>
+        <specular>1 1 1 1</specular>
+        <emissive>0 0 0 1</emissive>
+      </material>
+    </visual>
+  </gazebo>
   <joint
     name="rf_joint1"
@@ -338,5 +399,5 @@
       </geometry>
       <material
-        name="black">
+        name="white">
       </material>
     </visual>
@@ -351,4 +412,14 @@
     </collision>
   </link>
+  <gazebo reference="rf_link2">
+    <visual>
+      <material>
+        <ambient>1 1 1 1</ambient>
+        <diffuse>1 1 1 1</diffuse>
+        <specular>1 1 1 1</specular>
+        <emissive>0 0 0 1</emissive>
+      </material>
+    </visual>
+  </gazebo>
   <joint
     name="rf_joint2"
@@ -394,5 +465,5 @@
       </geometry>
       <material
-        name="black">
+        name="white">
       </material>
     </visual>
@@ -407,4 +478,14 @@
     </collision>
   </link>
+  <gazebo reference="lf_link1">
+    <visual>
+      <material>
+        <ambient>1 1 1 1</ambient>
+        <diffuse>1 1 1 1</diffuse>
+        <specular>1 1 1 1</specular>
+        <emissive>0 0 0 1</emissive>
+      </material>
+    </visual>
+  </gazebo>
   <joint
     name="lf_joint1"
@@ -450,5 +531,5 @@
       </geometry>
       <material
-        name="black">
+        name="white">
       </material>
     </visual>
@@ -463,4 +544,14 @@
     </collision>
   </link>
+  <gazebo reference="lf_link2">
+    <visual>
+      <material>
+        <ambient>1 1 1 1</ambient>
+        <diffuse>1 1 1 1</diffuse>
+        <specular>1 1 1 1</specular>
+        <emissive>0 0 0 1</emissive>
+      </material>
+    </visual>
+  </gazebo>
   <joint
     name="lf_joint2"
@@ -506,5 +597,5 @@
       </geometry>
       <material
-        name="black">
+        name="white">
       </material>
     </visual>
@@ -519,4 +610,14 @@
     </collision>
   </link>
+  <gazebo reference="camera_link">
+    <visual>
+      <material>
+        <ambient>1 1 1 1</ambient>
+        <diffuse>1 1 1 1</diffuse>
+        <specular>1 1 1 1</specular>
+        <emissive>0 0 0 1</emissive>
+      </material>
+    </visual>
+  </gazebo>
   <joint
     name="camera_joint"
@@ -676,3 +777,8 @@
       xyz="0 0 0" />
   </joint>
+  <gazebo>
+    <plugin name="gazebo_ros_control" filename="libgazebo_ros_control.so">
+      <robotNamespace>/puppy</robotNamespace>
+    </plugin>
+  </gazebo>
 </robot>

Commit message: add camera parameters

File: src/puppy_description/urdf/puppy.urdf.xacro (robot description, xacro)
@@ -782,3 +782,42 @@
     </plugin>
   </gazebo>
+  <!-- Add camera sensor macro -->
+  <xacro:macro name="camera_sensor" params="name parent_link">
+    <link name="${name}_link">
+      <visual>
+        <geometry>
+          <box size="0.1 0.1 0.1"/>
+        </geometry>
+        <material name="gray">
+          <color rgba="0.5 0.5 0.5 1"/>
+        </material>
+      </visual>
+    </link>
+    <joint name="${name}_joint" type="fixed">
+      <parent link="${parent_link}"/>
+      <child link="${name}_link"/>
+      <origin xyz="0 0 0.2" rpy="0 0 0"/>
+    </joint>
+    <gazebo reference="${name}_link">
+      <sensor type="camera" name="${name}_camera">
+        <update_rate>30</update_rate>
+        <camera>
+          <horizontal_fov>1.047</horizontal_fov>
+          <image>
+            <width>800</width>
+            <height>600</height>
+            <format>R8G8B8</format>
+          </image>
+          <clip>
+            <near>0.1</near>
+            <far>100</far>
+          </clip>
+        </camera>
+        <always_on>true</always_on>
+        <visualize>true</visualize>
+      </sensor>
+    </gazebo>
+  </xacro:macro>
+  <!-- Instantiate the camera sensor on a chosen link (e.g., head_link) -->
+  <xacro:camera_sensor name="head" parent_link="head_link"/>
 </robot>

Commit message: modify camera parameters

File: src/puppy_description/urdf/puppy.urdf.xacro (robot description, xacro)
@@ -619,4 +619,25 @@
       </material>
     </visual>
+    <sensor type="camera" name="head_camera_sensor">
+      <update_rate>30</update_rate>
+      <camera>
+        <horizontal_fov>1.39626</horizontal_fov>
+        <image>
+          <width>640</width>
+          <height>480</height>
+          <format>R8G8B8</format>
+        </image>
+        <clip>
+          <near>0.1</near>
+          <far>100</far>
+        </clip>
+      </camera>
+      <plugin name="gazebo_ros_camera" filename="libgazebo_ros_camera.so">
+        <cameraName>head_camera</cameraName>
+        <imageTopicName>image_raw</imageTopicName>
+        <cameraInfoTopicName>camera_info</cameraInfoTopicName>
+        <frameName>camera_link</frameName>
+      </plugin>
+    </sensor>
   </gazebo>
   <joint
@@ -782,10 +803,11 @@
     </plugin>
   </gazebo>
-  <!-- Add camera sensor macro -->
+  <!-- Updated camera sensor macro: using correct mesh for camera_link -->
   <xacro:macro name="camera_sensor" params="name parent_link">
     <link name="${name}_link">
       <visual>
         <geometry>
-          <box size="0.1 0.1 0.1"/>
+          <!-- Use the correct camera mesh -->
+          <mesh filename="package://puppy_description/meshes/camera_link.STL"/>
         </geometry>
         <material name="gray">
@@ -797,27 +819,8 @@
       <parent link="${parent_link}"/>
       <child link="${name}_link"/>
-      <origin xyz="0 0 0.2" rpy="0 0 0"/>
+      <origin xyz="0 0 0" rpy="0 0 0"/>
     </joint>
-    <gazebo reference="${name}_link">
-      <sensor type="camera" name="${name}_camera">
-        <update_rate>30</update_rate>
-        <camera>
-          <horizontal_fov>1.047</horizontal_fov>
-          <image>
-            <width>800</width>
-            <height>600</height>
-            <format>R8G8B8</format>
-          </image>
-          <clip>
-            <near>0.1</near>
-            <far>100</far>
-          </clip>
-        </camera>
-        <always_on>true</always_on>
-        <visualize>true</visualize>
-      </sensor>
-    </gazebo>
   </xacro:macro>
-  <!-- Instantiate the camera sensor on a chosen link (e.g., head_link) -->
-  <xacro:camera_sensor name="head" parent_link="head_link"/>
+  <!-- Instantiate the camera sensor -->
+  <xacro:camera_sensor name="head_camera" parent_link="camera_link"/>
 </robot>

Commit message: tilt camera and change parameters

File: src/puppy_description/urdf/puppy.urdf.xacro (robot description, xacro)
@@ -803,11 +803,10 @@
     </plugin>
   </gazebo>
-  <!-- Updated camera sensor macro: using correct mesh for camera_link -->
+  <!-- Updated camera sensor macro with a downward tilt -->
   <xacro:macro name="camera_sensor" params="name parent_link">
     <link name="${name}_link">
       <visual>
         <geometry>
-          <!-- Use the correct camera mesh -->
-          <mesh filename="package://puppy_description/meshes/camera_link.STL"/>
+          <box size="0.1 0.1 0.1"/>
         </geometry>
         <material name="gray">
@@ -819,6 +818,26 @@
       <parent link="${parent_link}"/>
       <child link="${name}_link"/>
-      <origin xyz="0 0 0" rpy="0 0 0"/>
+      <!-- Tilt camera downward (adjust pitch as needed) -->
+      <origin xyz="0 0 0.2" rpy="-0.5 0 0"/>
     </joint>
+    <gazebo reference="${name}_link">
+      <sensor type="camera" name="${name}_camera">
+        <update_rate>30</update_rate>
+        <camera>
+          <horizontal_fov>1.047</horizontal_fov>
+          <image>
+            <width>800</width>
+            <height>600</height>
+            <format>R8G8B8</format>
+          </image>
+          <clip>
+            <near>0.1</near>
+            <far>100</far>
+          </clip>
+        </camera>
+        <always_on>true</always_on>
+        <visualize>true</visualize>
+      </sensor>
+    </gazebo>
   </xacro:macro>
   <!-- Instantiate the camera sensor -->

Commit message: position camera to front and on location of camera mesh

File: src/puppy_description/urdf/puppy.urdf.xacro (robot description, xacro)
@@ -819,5 +819,5 @@
       <child link="${name}_link"/>
       <!-- Tilt camera downward (adjust pitch as needed) -->
-      <origin xyz="0 0 0.2" rpy="-0.5 0 0"/>
+      <origin xyz="0 0 0" rpy="0 0 -1.57"/>
     </joint>
     <gazebo reference="${name}_link">

Commit message: adjust camera positions to match both visual marker and feed

File: src/puppy_description/urdf/puppy.urdf.xacro (robot description, xacro)
@@ -572,86 +572,4 @@
       velocity="${motor_vec}" />
   </joint>
-  <link
-    name="camera_link">
-    <inertial>
-      <origin
-        xyz="7.8816314098059E-12 0.00830783337409231 -1.1027486424009E-09"
-        rpy="0 0 0" />
-      <mass
-        value="0.00255589783563972" />
-      <inertia
-        ixx="8.0750471256965E-08"
-        ixy="6.5213060632267E-17"
-        ixz="-9.04303283934642E-14"
-        iyy="7.57695997997755E-08"
-        iyz="1.85813457456822E-15"
-        izz="8.93985185103248E-08" />
-    </inertial>
-    <visual>
-      <origin
-        xyz="0 0 0"
-        rpy="0 0 0" />
-      <geometry>
-        <mesh
-          filename="package://puppy_description/meshes/camera_link.STL" />
-      </geometry>
-      <material
-        name="white">
-      </material>
-    </visual>
-    <collision>
-      <origin
-        xyz="0 0 0"
-        rpy="0 0 0" />
-      <geometry>
-        <mesh
-          filename="package://puppy_description/meshes/camera_link.STL" />
-      </geometry>
-    </collision>
-  </link>
-  <gazebo reference="camera_link">
-    <visual>
-      <material>
-        <ambient>1 1 1 1</ambient>
-        <diffuse>1 1 1 1</diffuse>
-        <specular>1 1 1 1</specular>
-        <emissive>0 0 0 1</emissive>
-      </material>
-    </visual>
-    <sensor type="camera" name="head_camera_sensor">
-      <update_rate>30</update_rate>
-      <camera>
-        <horizontal_fov>1.39626</horizontal_fov>
-        <image>
-          <width>640</width>
-          <height>480</height>
-          <format>R8G8B8</format>
-        </image>
-        <clip>
-          <near>0.1</near>
-          <far>100</far>
-        </clip>
-      </camera>
-      <plugin name="gazebo_ros_camera" filename="libgazebo_ros_camera.so">
-        <cameraName>head_camera</cameraName>
-        <imageTopicName>image_raw</imageTopicName>
-        <cameraInfoTopicName>camera_info</cameraInfoTopicName>
-        <frameName>camera_link</frameName>
-      </plugin>
-    </sensor>
-  </gazebo>
-  <joint
-    name="camera_joint"
-    type="fixed">
-    <origin
-      xyz="0 -0.100686660929431 0.017109543359257"
-      rpy="0.0342537604318887 0 0" />
-    <parent
-      link="base_link" />
-    <child
-      link="camera_link" />
-    <axis
-      xyz="0 0 0" />
-  </joint>
   <link name="lf_link3">
     <inertial>
@@ -803,5 +721,5 @@
     </plugin>
   </gazebo>
-  <!-- Updated camera sensor macro with a downward tilt -->
+  <!-- Updated camera sensor macro: remove duplicate "output" topic configuration -->
   <xacro:macro name="camera_sensor" params="name parent_link">
     <link name="${name}_link">
@@ -818,5 +736,5 @@
       <parent link="${parent_link}"/>
       <child link="${name}_link"/>
-      <!-- Tilt camera downward (adjust pitch as needed) -->
+      <!-- Tilt camera downward -->
       <origin xyz="0 0 0" rpy="0 0 -1.57"/>
     </joint>
@@ -838,8 +756,15 @@
         <always_on>true</always_on>
         <visualize>true</visualize>
+        <!-- Keep only one topic configuration -->
+        <plugin name="gazebo_ros_camera" filename="libgazebo_ros_camera.so">
+          <cameraName>head_camera</cameraName>
+          <imageTopicName>image_raw</imageTopicName>
+          <cameraInfoTopicName>camera_info</cameraInfoTopicName>
+          <frameName>${name}_link</frameName>
+        </plugin>
       </sensor>
     </gazebo>
   </xacro:macro>
-  <!-- Instantiate the camera sensor -->
-  <xacro:camera_sensor name="head_camera" parent_link="camera_link"/>
+  <!-- Ensure only one instantiation -->
+  <xacro:camera_sensor name="head_camera" parent_link="base_link"/>
 </robot>
