Commit message: fix dockerfile visual

File: puppy_ros2_ws/src/puppy_description/urdf/puppy.urdf.xacro (robot description, xacro)
@@ -1,6 +1,6 @@
 <?xml version="1.0" encoding="utf-8"?>
 <robot name="puppy" xmlns:xacro="http://ros.org/wiki/xacro">
-  <xacro:include filename="/workspace/src/puppy_description/urdf/puppy.transmission.xacro"/>
-  <xacro:include filename="/workspace/src/puppy_description/urdf/puppy.gazebo.xacro"/>
+  <xacro:include filename="puppy.transmission.xacro"/>
+  <xacro:include filename="puppy.gazebo.xacro"/>
   <xacro:include filename="materials.xacro" />
   <xacro:property name="motor_torque" value="0.5"/>
@@ -33,5 +33,5 @@
       <geometry>
         <mesh
-          filename="file:///workspace/models/puppybot/meshes/base_link.STL" />
+          filename="package://puppy_description/meshes/base_link.STL" />
       </geometry>
       <material
@@ -45,5 +45,5 @@
       <geometry>
         <mesh
-          filename="file:///workspace/models/puppybot/meshes/base_link.STL" />
+          filename="package://puppy_description/meshes/base_link.STL" />
       </geometry>
     </collision>
@@ -79,5 +79,5 @@
       <geometry>
         <mesh
-          filename="file:///workspace/models/puppybot/meshes/base_link.STL" />
+          filename="package://puppy_description/meshes/base_link.STL" />
       </geometry>
     </collision>
@@ -92,30 +92,30 @@
         value="0.0101534902703093" />
       <inertia
-        ixx="4.75129190044601E-06"
-        ixy="2.10473016237263E-08"
-        ixz="1.88925228411051E-08"
-        iyy="2.87659318790812E-06"
-        iyz="2.14913235084379E-06"
-        izz="2.92897619209419E-06" />
-    </inertial>
-    <visual>
-      <origin
-        xyz="0 0 0"
-        rpy="0 0 0" />
-      <geometry>
-        <mesh
-          filename="file:///workspace/models/puppybot/meshes/lb_link1.STL" />
-      </geometry>
-      <material
-        name="white">
-      </material>
-    </visual>
-    <collision>
-      <origin
-        xyz="0 0 0"
-        rpy="0 0 0" />
-      <geometry>
-        <mesh
-          filename="file:///workspace/models/puppybot/meshes/lb_link1.STL" />
+        ixx="0.0001015640290354"
+        ixy="5.44665608405109E-10"
+        ixz="-5.74905560030545E-09"
+        iyy="4.73014549137098E-05"
+        iyz="-4.46099046853099E-06"
+        izz="0.000137571042581761" />
+    </inertial>
+    <visual>
+      <origin
+        xyz="0 0 0"
+        rpy="0 0 0" />
+      <geometry>
+        <mesh
+          filename="package://puppy_description/meshes/lb_link1.STL" />
+      </geometry>
+      <material
+        name="blue">
+      </material>
+    </visual>
+    <collision>
+      <origin
+        xyz="0 0 0"
+        rpy="0 0 0" />
+      <geometry>
+        <mesh
+          filename="package://puppy_description/meshes/lb_link1.STL" />
       </geometry>
     </collision>
@@ -161,17 +161,17 @@
       <geometry>
         <mesh
-          filename="file:///workspace/models/puppybot/meshes/lb_link2.STL" />
-      </geometry>
-      <material
-        name="white">
-      </material>
-    </visual>
-    <collision>
-      <origin
-        xyz="0 0 0"
-        rpy="0 0 0" />
-      <geometry>
-        <mesh
-          filename="file:///workspace/models/puppybot/meshes/lb_link2.STL" />
+          filename="package://puppy_description/meshes/lb_link2.STL" />
+      </geometry>
+      <material
+        name="red">
+      </material>
+    </visual>
+    <collision>
+      <origin
+        xyz="0 0 0"
+        rpy="0 0 0" />
+      <geometry>
+        <mesh
+          filename="package://puppy_description/meshes/lb_link2.STL" />
       </geometry>
     </collision>
@@ -217,17 +217,17 @@
       <geometry>
         <mesh
-          filename="file:///workspace/models/puppybot/meshes/rb_link1.STL" />
-      </geometry>
-      <material
-        name="white">
-      </material>
-    </visual>
-    <collision>
-      <origin
-        xyz="0 0 0"
-        rpy="0 0 0" />
-      <geometry>
-        <mesh
-          filename="file:///workspace/models/puppybot/meshes/rb_link1.STL" />
+          filename="package://puppy_description/meshes/rb_link1.STL" />
+      </geometry>
+      <material
+        name="blue">
+      </material>
+    </visual>
+    <collision>
+      <origin
+        xyz="0 0 0"
+        rpy="0 0 0" />
+      <geometry>
+        <mesh
+          filename="package://puppy_description/meshes/rb_link1.STL" />
       </geometry>
     </collision>
@@ -273,17 +273,17 @@
       <geometry>
         <mesh
-          filename="file:///workspace/models/puppybot/meshes/rb_link2.STL" />
-      </geometry>
-      <material
-        name="white">
-      </material>
-    </visual>
-    <collision>
-      <origin
-        xyz="0 0 0"
-        rpy="0 0 0" />
-      <geometry>
-        <mesh
-          filename="file:///workspace/models/puppybot/meshes/rb_link2.STL" />
+          filename="package://puppy_description/meshes/rb_link2.STL" />
+      </geometry>
+      <material
+        name="red">
+      </material>
+    </visual>
+    <collision>
+      <origin
+        xyz="0 0 0"
+        rpy="0 0 0" />
+      <geometry>
+        <mesh
+          filename="package://puppy_description/meshes/rb_link2.STL" />
       </geometry>
     </collision>
@@ -329,17 +329,17 @@
       <geometry>
         <mesh
-          filename="file:///workspace/models/puppybot/meshes/rf_link1.STL" />
-      </geometry>
-      <material
-        name="white">
-      </material>
-    </visual>
-    <collision>
-      <origin
-        xyz="0 0 0"
-        rpy="0 0 0" />
-      <geometry>
-        <mesh
-          filename="file:///workspace/models/puppybot/meshes/rf_link1.STL" />
+          filename="package://puppy_description/meshes/rf_link1.STL" />
+      </geometry>
+      <material
+        name="blue">
+      </material>
+    </visual>
+    <collision>
+      <origin
+        xyz="0 0 0"
+        rpy="0 0 0" />
+      <geometry>
+        <mesh
+          filename="package://puppy_description/meshes/rf_link1.STL" />
       </geometry>
     </collision>
@@ -385,17 +385,17 @@
       <geometry>
         <mesh
-          filename="file:///workspace/models/puppybot/meshes/rf_link2.STL" />
-      </geometry>
-      <material
-        name="white">
-      </material>
-    </visual>
-    <collision>
-      <origin
-        xyz="0 0 0"
-        rpy="0 0 0" />
-      <geometry>
-        <mesh
-          filename="file:///workspace/models/puppybot/meshes/rf_link2.STL" />
+          filename="package://puppy_description/meshes/rf_link2.STL" />
+      </geometry>
+      <material
+        name="red">
+      </material>
+    </visual>
+    <collision>
+      <origin
+        xyz="0 0 0"
+        rpy="0 0 0" />
+      <geometry>
+        <mesh
+          filename="package://puppy_description/meshes/rf_link2.STL" />
       </geometry>
     </collision>
@@ -441,17 +441,17 @@
       <geometry>
         <mesh
-          filename="file:///workspace/models/puppybot/meshes/lf_link1.STL" />
-      </geometry>
-      <material
-        name="white">
-      </material>
-    </visual>
-    <collision>
-      <origin
-        xyz="0 0 0"
-        rpy="0 0 0" />
-      <geometry>
-        <mesh
-          filename="file:///workspace/models/puppybot/meshes/lf_link1.STL" />
+          filename="package://puppy_description/meshes/lf_link1.STL" />
+      </geometry>
+      <material
+        name="blue">
+      </material>
+    </visual>
+    <collision>
+      <origin
+        xyz="0 0 0"
+        rpy="0 0 0" />
+      <geometry>
+        <mesh
+          filename="package://puppy_description/meshes/lf_link1.STL" />
       </geometry>
     </collision>
@@ -497,17 +497,17 @@
       <geometry>
         <mesh
-          filename="file:///workspace/models/puppybot/meshes/lf_link2.STL" />
-      </geometry>
-      <material
-        name="white">
-      </material>
-    </visual>
-    <collision>
-      <origin
-        xyz="0 0 0"
-        rpy="0 0 0" />
-      <geometry>
-        <mesh
-          filename="file:///workspace/models/puppybot/meshes/lf_link2.STL" />
+          filename="package://puppy_description/meshes/lf_link2.STL" />
+      </geometry>
+      <material
+        name="red">
+      </material>
+    </visual>
+    <collision>
+      <origin
+        xyz="0 0 0"
+        rpy="0 0 0" />
+      <geometry>
+        <mesh
+          filename="package://puppy_description/meshes/lf_link2.STL" />
       </geometry>
     </collision>
@@ -553,17 +553,17 @@
       <geometry>
         <mesh
-          filename="file:///workspace/models/puppybot/meshes/camera_link.STL" />
-      </geometry>
-      <material
-        name="white">
-      </material>
-    </visual>
-    <collision>
-      <origin
-        xyz="0 0 0"
-        rpy="0 0 0" />
-      <geometry>
-        <mesh
-          filename="file:///workspace/models/puppybot/meshes/camera_link.STL" />
+          filename="package://puppy_description/meshes/camera_link.STL" />
+      </geometry>
+      <material
+        name="black">
+      </material>
+    </visual>
+    <collision>
+      <origin
+        xyz="0 0 0"
+        rpy="0 0 0" />
+      <geometry>
+        <mesh
+          filename="package://puppy_description/meshes/camera_link.STL" />
       </geometry>
     </collision>

Commit message: testing rviz integration into main pipeline

File: puppy_ros2_ws/src/puppy_description/urdf/puppy.urdf.xacro (robot description, xacro)
@@ -726,3 +726,49 @@
       xyz="0 0 0" />
   </joint>
+  <!-- ros2_control hardware interface -->
+  <ros2_control name="GazeboSystem" type="system">
+    <hardware>
+      <plugin>gazebo_ros2_control/GazeboSystem</plugin>
+    </hardware>
+    <joint name="lf_joint1">
+      <command_interface name="position"/>
+      <state_interface name="position"/>
+      <state_interface name="velocity"/>
+    </joint>
+    <joint name="lf_joint2">
+      <command_interface name="position"/>
+      <state_interface name="position"/>
+      <state_interface name="velocity"/>
+    </joint>
+    <joint name="lb_joint1">
+      <command_interface name="position"/>
+      <state_interface name="position"/>
+      <state_interface name="velocity"/>
+    </joint>
+    <joint name="lb_joint2">
+      <command_interface name="position"/>
+      <state_interface name="position"/>
+      <state_interface name="velocity"/>
+    </joint>
+    <joint name="rf_joint1">
+      <command_interface name="position"/>
+      <state_interface name="position"/>
+      <state_interface name="velocity"/>
+    </joint>
+    <joint name="rf_joint2">
+      <command_interface name="position"/>
+      <state_interface name="position"/>
+      <state_interface name="velocity"/>
+    </joint>
+    <joint name="rb_joint1">
+      <command_interface name="position"/>
+      <state_interface name="position"/>
+      <state_interface name="velocity"/>
+    </joint>
+    <joint name="rb_joint2">
+      <command_interface name="position"/>
+      <state_interface name="position"/>
+      <state_interface name="velocity"/>
+    </joint>
+  </ros2_control>
 </robot>
