Commit message: fix controller issues

File: puppy_ros2_ws/src/puppy_description/urdf/puppy.gazebo.xacro (robot description, xacro)
@@ -1,4 +1,12 @@
 <?xml version="1.0"?>
 <robot name="puppy" xmlns:xacro="http://www.ros.org/wiki/xacro">
+  <!-- Gazebo Control Plugin -->
+  <gazebo>
+    <plugin filename="libgz_ros2_control-system.so" name="gz_ros2_control::GazeboSimROS2ControlPlugin">
+      <robot_param>robot_description</robot_param>
+      <robot_param_node>robot_state_publisher</robot_param_node>
+      <parameters>$(find puppy_description)/config/ros2_control.yaml</parameters>
+    </plugin>
+  </gazebo>
   <xacro:macro name="model_color" params="link_name">
     <gazebo reference="${link_name}">

File: puppy_ros2_ws/src/puppy_description/urdf/puppy.transmission.xacro (robot description, xacro)
@@ -3,7 +3,9 @@
   <!-- ROS2 Control transmission format -->
   <!-- Define ros2_control tag for the robot -->
-  <ros2_control name="PuppyHardware" type="system">
+  <ros2_control name="gazebo_hardware" type="gz_ros2_control/GazeboSimSystem">
     <hardware>
-      <plugin>gazebo_ros2_control/GazeboSystem</plugin>
+      <plugin>gz_ros2_control/GazeboSimSystem</plugin>
+      <param name="robot_description">robot_description</param>
+      <param name="robot_param_node">robot_state_publisher</param>
     </hardware>
     <!-- ROS2 Control Joint configuration -->
@@ -11,6 +13,4 @@
       <joint name="${joint_name}">
         <command_interface name="position"/>
-        <command_interface name="velocity"/>
-        <command_interface name="effort"/>
         <state_interface name="position"/>
         <state_interface name="velocity"/>
@@ -28,24 +28,3 @@
     <xacro:joint_control joint_name="rb_joint2"/>
   </ros2_control>
-  <!-- Legacy transmission blocks for compatibility -->
-  <xacro:macro name="transmission_block" params="joint_name">
-    <transmission name="${joint_name}_trans">
-      <type>transmission_interface/SimpleTransmission</type>
-      <joint name="${joint_name}">
-        <hardwareInterface>hardware_interface/EffortJointInterface</hardwareInterface>
-      </joint>
-      <actuator name="${joint_name}_motor">
-        <hardwareInterface>hardware_interface/EffortJointInterface</hardwareInterface>
-        <mechanicalReduction>1</mechanicalReduction>
-      </actuator>
-    </transmission>
-  </xacro:macro>
-  <xacro:transmission_block joint_name="lf_joint1"/>
-  <xacro:transmission_block joint_name="lf_joint2"/>
-  <xacro:transmission_block joint_name="lb_joint1"/>
-  <xacro:transmission_block joint_name="lb_joint2"/>
-  <xacro:transmission_block joint_name="rf_joint1"/>
-  <xacro:transmission_block joint_name="rf_joint2"/>
-  <xacro:transmission_block joint_name="rb_joint1"/>
-  <xacro:transmission_block joint_name="rb_joint2"/>
 </robot>
